Commit message: fix motion nodes

File: simulation_ws/src/osr_urdf_with_controllers_and_launch/rover_description/urdf/rover_description.urdf (robot description, URDF)
Before this commit: robot rover_description, 16 links, 15 joints
Joints:
- joint camera_joint: origin xyz=1 0 1 rpy=0 0 0 -> xyz=1 0 1 rpy=0 0 3.14

Commit message: fixed urdf, added sensors to urdf, fixed launchfile

File: simulation_ws/src/osr_urdf_with_controllers_and_launch/rover_description/urdf/rover_description.urdf (robot description, URDF)
Before this commit: robot rover_description, 16 links, 15 joints
Links:
- added link depthcamera_link; collision box size=0.01 0.01 0.01
- added link imu_link
- added link imu_wheel_lb_link
- added link imu_wheel_lf_link
- added link imu_wheel_lm_link
- added link imu_wheel_rb_link
- added link imu_wheel_rf_link
- added link imu_wheel_rm_link
- added link pointcloud_link
- link camera_link: geometry collision box size=0.01 0.01 0.01
Joints:
- added joint depthcamera_joint: type fixed, parent body, child depthcamera_link, origin xyz=-0.1 0 0 rpy=0 0 3.14, axis 0 0 0
- added joint imu_joint: type fixed, parent body, child imu_link, origin xyz=-0.032 0 0.068 rpy=0 0 3.14
- added joint imu_wheel_lb_joint: type fixed, parent corner_lb, child imu_wheel_lb_link, origin xyz=0.04 -0.069 0.005 rpy=-1.58 0 0
- added joint imu_wheel_lf_joint: type fixed, parent corner_lf, child imu_wheel_lf_link, origin xyz=0.028 -0.089 0.01 rpy=-1.58 0 0
- added joint imu_wheel_lm_joint: type fixed, parent bogie_left, child imu_wheel_lm_link, origin xyz=0.105 -0.179 0.078 rpy=-1.58 0 0
- added joint imu_wheel_rb_joint: type fixed, parent corner_rb, child imu_wheel_rb_link, origin xyz=0 -0.1 0 rpy=-1.58 0 0
- added joint imu_wheel_rf_joint: type fixed, parent corner_rf, child imu_wheel_rf_link, origin xyz=0 -0.1 0 rpy=-1.58 0 0
- added joint imu_wheel_rm_joint: type fixed, parent bogie_right, child imu_wheel_rm_link, origin xyz=0.066 -0.182 -0.079 rpy=-1.58 0 0
- added joint pointcloud_joint: type fixed, parent depthcamera_link, child pointcloud_link, origin xyz=-0.1 0 0 rpy=-1.58 0 -1.58, axis 0 0 0
- joint body_rocker_left: axis 1  0  0 -> 0  1  0
- joint body_rocker_right: axis 0  0 -1 -> 0  0  -1
- joint camera_joint: origin xyz=1 0 1 rpy=0 0 3.14 -> xyz=-0.1 0 0 rpy=0 0 3.14

Commit message: Port rover description from JPL project

File: simulation_ws/src/osr_urdf_with_controllers_and_launch/rover_description/urdf/rover_description.urdf (robot description, URDF)
Before this commit: robot rover_description, 25 links, 24 joints
Links:
- added link base_scan
- link body: geometry collision mesh filename=package://rover_description/meshes/body.STL scale=1 1 1; visual mesh filename=package://rover_description/meshes/body.dae scale=1 1 1
- link bogie_left: geometry collision mesh filename=package://rover_description/meshes/bogie_left.STL scale=1 1 1; visual mesh filename=package://rover_description/meshes/bogie_left.dae scale=1 1 1
- link bogie_right: geometry collision mesh filename=package://rover_description/meshes/bogie_right.STL scale=1 1 1; visual mesh filename=package://rover_description/meshes/bogie_right.dae scale=1 1 1
- link corner_lb: geometry collision mesh filename=package://rover_description/meshes/corner_lb.STL scale=1 1 1; visual mesh filename=package://rover_description/meshes/corner_lb.dae scale=1 1 1
- link corner_lf: geometry collision mesh filename=package://rover_description/meshes/corner_lf.STL scale=1 1 1; visual mesh filename=package://rover_description/meshes/corner_lf.dae scale=1 1 1
- link corner_rb: geometry collision mesh filename=package://rover_description/meshes/corner_rb.STL scale=1 1 1; visual mesh filename=package://rover_description/meshes/corner_rb.dae scale=1 1 1
- link corner_rf: geometry collision mesh filename=package://rover_description/meshes/corner_rf.STL scale=1 1 1; visual mesh filename=package://rover_description/meshes/corner_rf.dae scale=1 1 1
- link rocker_left: geometry collision mesh filename=package://rover_description/meshes/rocker_left.STL scale=1 1 1; visual mesh filename=package://rover_description/meshes/rocker_left.dae scale=1 1 1
- link rocker_right: geometry collision mesh filename=package://rover_description/meshes/rocker_right.STL scale=1 1 1; visual mesh filename=package://rover_description/meshes/rocker_right.dae scale=1 1 1
- link wheel_lb: geometry collision mesh filename=package://rover_description/meshes/wheel_lb.STL scale=1 1 1; visual mesh filename=package://rover_description/meshes/wheel_lb.dae scale=1 1 1
- link wheel_lf: geometry collision mesh filename=package://rover_description/meshes/wheel_lf.STL scale=1 1 1; visual mesh filename=package://rover_description/meshes/wheel_lf.dae scale=1 1 1
- link wheel_lm: geometry collision mesh filename=package://rover_description/meshes/wheel_lm.STL scale=1 1 1; visual mesh filename=package://rover_description/meshes/wheel_lm.dae scale=1 1 1
- link wheel_rb: geometry collision mesh filename=package://rover_description/meshes/wheel_rb.STL scale=1 1 1; visual mesh filename=package://rover_description/meshes/wheel_rb.dae scale=1 1 1
- link wheel_rf: geometry collision mesh filename=package://rover_description/meshes/wheel_rf.STL scale=1 1 1; visual mesh filename=package://rover_description/meshes/wheel_rf.dae scale=1 1 1
- link wheel_rm: geometry collision mesh filename=package://rover_description/meshes/wheel_rm.STL scale=1 1 1; visual mesh filename=package://rover_description/meshes/wheel_rm.dae scale=1 1 1
Joints:
- added joint scan_joint: type fixed, parent body, child base_scan, origin xyz=-.075 0.03 -.075 rpy=0 -0.275 0
